File: dock/kicad/ESP32-Bit-Pirate.kicad_sch (KiCad schematic)
At the start: 18 parts, among them CN1 HX25418-10WA, J1 Conn_01x22, J2 Conn_01x22, J3 Conn_01x10V, J4 Conn_01x22, J5 Conn_01x22, J6 Conn_01x22, J7 Conn_02x03, U1 ESP32-S3-DEVKITC-1-N8R2, U2 TLV75518PDBV

Commit message: Added new name for kicad project
Other:
- note added: "ESP32 Bit Pirate Dock"
- note removed: "ESP32 Bus Pirate Dock"
- company: ESP32 Bus Pirate -> ESP32 Bit Pirate
- title: ESP32 Bus Pirate Dock -> ESP32 Bit Pirate Dock
