File: dock/kicad/voltage_level_translator.kicad_sch (KiCad schematic)
At the start: 29 parts, among them J8 TC2050, Q1 2SK2009, SW1 TA-3532S-A2, U3 TS5A3157DBVR, U4 TXS0108EPW, U5 TXS0108EPW, U6 TMUX1574PW, U7 TMUX1574PW

Commit message: Added new name for kicad project
Other:
- title: (none) -> ESP32 Bit Pirate Dock
