File: dock/kicad/ESP32-Bus-Pirate-Dock.kicad_sch (KiCad schematic)
At the start: 18 parts, among them CN1 HX25418-10WA, J1 Conn_01x22, J2 Conn_01x22, J3 Conn_01x10V, J4 Conn_01x22, J5 Conn_01x22, J6 Conn_01x22, J7 Conn_02x03, U1 ESP32-S3-DEVKITC-1-N8R2, U2 TLV75518PDBV

Commit message: Renamed project files with new name
Other:
- company: ESP32 Bus Pirate -> ESP32 Bus Pirate Team
