File: dock/kicad/ESP32-Bit-Pirate-Dock.kicad_pcb (KiCad board)
At the start: 4 copper layers, 80 x 73.8 mm, 49 parts, among them CN1 HX25418-10WA, J1 Conn_01x22, J2 Conn_01x22, J3 Conn_01x10V, J4 Conn_01x22, J5 Conn_01x22, J6 Conn_01x22, J7 Conn_02x03, J8 TC2050, Q1 2SK2009, SW1 TA-3532S-A2, U2 TLV75518PDBV, U3 TS5A3157DBVR, U4 TXS0108EPW, U5 TXS0108EPW, U6 TMUX1574PW, U7 TMUX1574PW

Commit message: Fixed file names & added logo library
Co-Authored-By: fdufnews <fdufnews@free.fr>
Parts:
- G***: value LOGO -> ESP32-Bit-Pirate-Logo-Dock; footprint LOGO -> ESP32-Bit-Pirate-Logo:ESP32-Bit-Pirate-Logo-Dock
Changed lines of the file:
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@@
 		(embedded_fonts no)
 	)
-	(footprint "LOGO"
+	(footprint "ESP32-Bit-Pirate-Logo:ESP32-Bit-Pirate-Logo-Dock"
 		(layer "F.Cu")
 		(at 76.5 136.5)
@@
 			)
 		)
-		(property "Value" "LOGO"
+		(property "Value" "ESP32-Bit-Pirate-Logo-Dock"
 			(at 0.75 0 0)
 			(layer "F.SilkS")
