File: c5_adapter/kicad/c5_adapter.kicad_pcb (KiCad board)
At the start: 4 copper layers, 50 x 45 mm, 7 parts, among them J1 Conn_01x10, J3 Conn_01x16, J4 Conn_01x16, J5 Conn_01x16, J6 Conn_01x16, SW1 MK-12C02-G020

Commit message: Changed stackup to 2 layers
Routing:
- removed copper zone on In1.Cu, net GND
- removed copper zone on In2.Cu, net GND
Other:
- copper layers 4 -> 2
Changed lines of the file:
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@@
 	(layers
 		(0 "F.Cu" signal)
-		(4 "In1.Cu" power)
-		(6 "In2.Cu" mixed)
 		(2 "B.Cu" signal)
 		(13 "F.Paste" user)
@@
 			)
 			(layer "dielectric 1"
-				(type "prepreg")
-				(thickness 0.1)
-				(material "FR4")
-				(epsilon_r 4.5)
-				(loss_tangent 0.02)
-			)
-			(layer "In1.Cu"
-				(type "copper")
-				(thickness 0.035)
-			)
-			(layer "dielectric 2"
 				(type "core")
-				(thickness 1.24)
-				(material "FR4")
-				(epsilon_r 4.5)
-				(loss_tangent 0.02)
-			)
-			(layer "In2.Cu"
-				(type "copper")
-				(thickness 0.035)
-			)
-			(layer "dielectric 3"
-				(type "prepreg")
-				(color "#808080FF")
-				(thickness 0.1)
+				(thickness 1.51)
 				(material "FR4")
 				(epsilon_r 4.5)
@@
 	)
 	(zone
-		(layers "F.Cu" "B.Cu" "In1.Cu" "F.SilkS" "In2.Cu")
+		(net "GND")
+		(layers "F.Cu" "B.Cu")
+		(hatch edge 0.5)
+		(connect_pads
+			(clearance 0.4)
+		)
+		(min_thickness 0.25)
+		(fill yes
+			(thermal_gap 0.5)
+			(thermal_bridge_width 0.5)
+			(island_removal_mode 0)
+		)
+		(polygon
+			(pts
+				(xy 172.5 78.4) (xy 223.8 78.4) (xy 223.8 124.7) (xy 172.7 124.7)
+			)
+		)
+	)
+	(zone
+		(layers "F.Cu" "B.Cu" "F.SilkS")
 		(name "Antennaa Keep Out")
 		(hatch edge 0.5)
@@
 			)
 		)
-	)
-	(zone
-		(net "GND")
-		(layers "F.Cu" "B.Cu" "In1.Cu" "In2.Cu")
-		(hatch edge 0.5)
-		(connect_pads
-			(clearance 0.4)
-		)
-		(min_thickness 0.25)
-		(fill yes
-			(thermal_gap 0.5)
-			(thermal_bridge_width 0.5)
-			(island_removal_mode 0)
-		)
-		(polygon
-			(pts
-				(xy 172.5 78.4) (xy 223.8 78.4) (xy 223.8 124.7) (xy 172.7 124.7)
-			)
-		)
