File: c5_adapter/kicad/c5_adapter.kicad_sch (KiCad schematic)
At the start: 10 parts, among them J1 Conn_01x10, J2 Conn_01x10, J3 Conn_01x16, J4 Conn_01x16, J5 Conn_01x16, J6 Conn_01x16, SW1 MK-12C02-G020, U1 ESP32-C5-DevKitC-1

Commit message: Changed stackup to 2 layers
Parts:
- removed D1: LED, LED_SMD:LED_0805_2012Metric, symbol Device:LED
- removed R1: 1k, Resistor_SMD:R_0805_2012Metric, symbol Device:R
