File: MCU_adapters/stamps3_adapter/stamps3_adapter.kicad_sch (KiCad schematic)
At the start: 5 parts, among them J1 Conn_01x22, J2 Conn_01x22, J3 Conn_01x09_Socket, J4 Conn_01x06_Socket

Commit message: Updated adapters with USB logo
Added an USB logo to ensure the card is inserted the right way up.
Added an USB logo in the logo library
Updated the gerber files
Parts:
- added G2: (no value), logo:LOGO_USB, symbol logo:LOGO_USB
Changed lines of the file:
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@@
+	)
+	(symbol
+		(lib_id "logo:LOGO_USB")
+		(at 68.58 165.1 0)
+		(unit 1)
+		(body_style 1)
+		(exclude_from_sim no)
+		(in_bom no)
+		(on_board yes)
+		(in_pos_files yes)
+		(dnp no)
+		(fields_autoplaced yes)
+		(property "Reference" "G2"
+			(at 75.565 168.1692 0)
+			(show_name no)
+			(do_not_autoplace no)
+			(effects
+				(font
+					(size 1.27 1.27)
+				)
+				(justify left)
+			)
+		)
+		(property "Value" ""
+			(at 68.58 165.1 0)
+			(show_name no)
+			(do_not_autoplace no)
+			(effects
+				(font
+					(size 1.27 1.27)
+				)
+			)
+		)
+		(property "Footprint" "logo:LOGO_USB"
+			(at 68.58 165.1 0)
+			(hide yes)
+			(show_name no)
+			(do_not_autoplace no)
+			(effects
+				(font
+					(size 1.27 1.27)
+				)
+			)
+		)
+		(property "Datasheet" ""
+			(at 68.58 165.1 0)
+			(hide yes)
+			(show_name no)
+			(do_not_autoplace no)
+			(effects
+				(font
+					(size 1.27 1.27)
+				)
+			)
+		)
+		(property "Description" ""
+			(at 68.58 165.1 0)
+			(hide yes)
+			(show_name no)
+			(do_not_autoplace no)
+			(effects
+				(font
+					(size 1.27 1.27)
+				)
+			)
+		)
+		(instances
+			(project "stamps3_adapter"
+				(path "/59c5a8d0-1c3e-4465-8c7d-6fc2dddcf807"
+					(reference "G2")
+					(unit 1)
+				)
+			)
+		)
 	)
 	(symbol
