File: MCU_adapters/wifilorav4_adapter/wifilorav4_adapter.kicad_pcb (KiCad board)
At the start: 2 copper layers, 34.4 x 57.1 mm, 5 parts, among them J1 Conn_01x22, J2 Conn_01x22, J3 Conn_01x18_Socket, J4 Conn_01x18_Socket

Commit message: Updated adapters with USB logo
Added an USB logo to ensure the card is inserted the right way up.
Added an USB logo in the logo library
Updated the gerber files
Parts:
- added G2: ~, logo:LOGO_USB, F.Cu at (91.8, 70.6)
- moved G1 42.2 mm to (91.9, 35.2)
Changed lines of the file:
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@@
 		)
+	)
+	(footprint "logo:LOGO_USB"
+		(layer "F.Cu")
+		(at 91.8 70.63)
+		(property "Reference" "G2"
+			(at 0 -0.5 0)
+			(unlocked yes)
+			(layer "F.SilkS")
+			(hide yes)
+			(effects
+				(font
+					(size 1 1)
+					(thickness 0.15)
+				)
+			)
+		)
+		(property "Value" "~"
+			(at 0 1 0)
+			(unlocked yes)
+			(layer "F.Fab")
+			(effects
+				(font
+					(size 1 1)
+					(thickness 0.15)
+				)
+			)
+		)
+		(property "Datasheet" ""
+			(at 0 0 0)
+			(unlocked yes)
+			(layer "F.Fab")
+			(hide yes)
+			(effects
+				(font
+					(size 1 1)
+					(thickness 0.15)
+				)
+			)
+		)
+		(property "Description" ""
+			(at 0 0 0)
+			(unlocked yes)
+			(layer "F.Fab")
+			(hide yes)
+			(effects
+				(font
+					(size 1 1)
+					(thickness 0.15)
+				)
+			)
+		)
+		(sheetname "/")
+		(sheetfile "wifilorav4_adapter.kicad_sch")
+		(units
+			(unit
+				(name "A")
+				(pins)
+			)
+		)
+		(attr smd exclude_from_bom)
+		(duplicate_pad_numbers_are_jumpers no)
+		(fp_rect
+			(start -5.08 0)
+			(end 3.81 5.08)
+			(stroke
+				(width 0.3)
+				(type solid)
+			)
+			(fill no)
+			(layer "F.SilkS")
+		)
+		(fp_text user "USB"
+			(at -5.08 8.89 0)
+			(unlocked yes)
+			(layer "F.SilkS")
+			(effects
+				(font
+					(size 2.54 2.4)
+					(thickness 0.25)
+				)
+				(justify left bottom)
+			)
+		)
+		(fp_text user "${REFERENCE}"
+			(at 0 2.5 0)
+			(unlocked yes)
+			(layer "F.Fab")
+			(effects
+				(font
+					(size 1 1)
+					(thickness 0.15)
+				)
+			)
+		)
+		(embedded_fonts no)
 	)
 	(footprint "Connector_PinSocket_2.54mm:PinSocket_1x18_P2.54mm_Vertical"
@@
 	(footprint "logo:logoBP"
 		(layer "F.Cu")
-		(at 91.9226 77.47)
+		(at 91.868872 35.242152)
 		(property "Reference" "G1"
 			(at 0 -0.5 0)
